File: ROG_Condor.brd (EAGLE design)
At the start: 45.4 x 44.4 mm, 35 parts, among them IC1 TL072P, IC2 TL072P, Q1 J201

Commit message: Version 1.0 with layout sent to OSHPark
Parts:
- C1, C2, C3: value 0.047uF -> 47nF
- C5: value 0.001uF -> 1nF
- C6: value 0.015uF -> 15nF
- C7, C8: value 0.0039uF -> 3.9nF
- renumbered +9V1 to +9V, GND1 to GND, IN1 to IN, OUT1 to OUT
Other:
- board text added: "ROG Condor Cabsim"
- board text added: "Xenocoder Pedals v1.0 01.2017"
