File: ROG_Condor.sch (EAGLE design)
At the start: 35 parts, among them IC1 TL072P, IC2 TL072P, Q1 J201

Commit message: Version 1.0 with layout sent to OSHPark
Parts:
- C1, C2, C3: value 0.047uF -> 47nF
- C5: value 0.001uF -> 1nF
- C6: value 0.015uF -> 15nF
- C7, C8: value 0.0039uF -> 3.9nF
- renumbered +9V1 to +9V, GND1 to GND, IN1 to IN, OUT1 to OUT
Changed lines of the file:
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@@
 <part name="R16" library="mb_resistors" deviceset="6MM" device=".3" value="22k"/>
 <part name="R17" library="mb_resistors" deviceset="6MM" device=".3" value="100k"/>
-<part name="+9V1" library="mb_supply" deviceset="+9V(T)" device=""/>
-<part name="GND1" library="mb_supply" deviceset="GND(T)" device=""/>
+<part name="+9V" library="mb_supply" deviceset="+9V(T)" device=""/>
+<part name="GND" library="mb_supply" deviceset="GND(T)" device=""/>
 <part name="GND3" library="mb_supply" deviceset="GND" device=""/>
 <part name="GND4" library="mb_supply" deviceset="GND" device=""/>
 <part name="GND5" library="mb_supply" deviceset="GND" device=""/>
 <part name="GND6" library="mb_supply" deviceset="GND" device=""/>
-<part name="IN1" library="mb_supply" deviceset="IN(T)" device=""/>
-<part name="OUT1" library="mb_supply" deviceset="OUT(T)" device=""/>
+<part name="IN" library="mb_supply" deviceset="IN(T)" device=""/>
+<part name="OUT" library="mb_supply" deviceset="OUT(T)" device=""/>
 <part name="LED" library="mb_supply" deviceset="PAD" device="" value="LED"/>
 <part name="D1" library="mb_diodes" deviceset="LED" device="3MM"/>
-<part name="C1" library="mb_caps-chicklet" deviceset="075X040" device="2" value="0.047uF"/>
-<part name="C2" library="mb_caps-chicklet" deviceset="075X040" device="2" value="0.047uF"/>
-<part name="C3" library="mb_caps-chicklet" deviceset="075X040" device="2" value="0.047uF"/>
+<part name="C1" library="mb_caps-chicklet" deviceset="075X040" device="2" value="47nF"/>
+<part name="C2" library="mb_caps-chicklet" deviceset="075X040" device="2" value="47nF"/>
+<part name="C3" library="mb_caps-chicklet" deviceset="075X040" device="2" value="47nF"/>
 <part name="TRIM" library="mb_pots" deviceset="POT" device="TRIM" value="100k"/>
 <part name="Q1" library="mb_trans" deviceset="J201" device=""/>
@@
 <part name="C4" library="mb_caps-electro" deviceset="050" device="1" value="22uF"/>
 <part name="VA1" library="mb_supply" deviceset="VA" device=""/>
-<part name="C5" library="mb_caps-chicklet" deviceset="075X040" device="2" value="0.001uF"/>
-<part name="C6" library="mb_caps-chicklet" deviceset="075X040" device="2" value="0.015uF"/>
+<part name="C5" library="mb_caps-chicklet" deviceset="075X040" device="2" value="1nF"/>
+<part name="C6" library="mb_caps-chicklet" deviceset="075X040" device="2" value="15nF"/>
 <part name="IC1" library="mb_ics" deviceset="TL072" device="P"/>
 <part name="IC2" library="mb_ics" deviceset="TL072" device="P"/>
 <part name="VA2" library="mb_supply" deviceset="VA" device=""/>
-<part name="C7" library="mb_caps-chicklet" deviceset="075X040" device="2" value="0.0039uF"/>
+<part name="C7" library="mb_caps-chicklet" deviceset="075X040" device="2" value="3.9nF"/>
 <part name="VA3" library="mb_supply" deviceset="VA" device=""/>
 <part name="GND10" library="mb_supply" deviceset="GND" device=""/>
-<part name="C8" library="mb_caps-chicklet" deviceset="075X040" device="2" value="0.0039uF"/>
+<part name="C8" library="mb_caps-chicklet" deviceset="075X040" device="2" value="3.9nF"/>
 <part name="C9" library="mb_caps-electro" deviceset="050" device="1" value="22uF"/>
 <part name="GND12" library="mb_supply" deviceset="GND" device=""/>
@@
 <instance part="R16" gate="G$1" x="142.24" y="55.88" rot="R180"/>
 <instance part="R17" gate="G$1" x="119.38" y="91.44" rot="R90"/>
-<instance part="+9V1" gate="+9V" x="-7.62" y="68.58" rot="R90"/>
-<instance part="GND1" gate="GND" x="12.7" y="45.72"/>
+<instance part="+9V" gate="+9V" x="-7.62" y="68.58" rot="R90"/>
+<instance part="GND" gate="GND" x="12.7" y="45.72"/>
 <instance part="GND3" gate="GND" x="33.02" y="45.72"/>
 <instance part="GND4" gate="GND" x="43.18" y="45.72"/>
 <instance part="GND5" gate="GND" x="78.74" y="83.82"/>
 <instance part="GND6" gate="GND" x="55.88" y="66.04"/>
-<instance part="IN1" gate="G$1" x="-7.62" y="83.82"/>
-<instance part="OUT1" gate="G$1" x="193.04" y="48.26"/>
+<instance part="IN" gate="G$1" x="-7.62" y="83.82"/>
+<instance part="OUT" gate="G$1" x="193.04" y="48.26"/>
 <instance part="LED" gate="G$1" x="0" y="35.56" rot="R270"/>
 <instance part="D1" gate="G$1" x="0" y="45.72" rot="R90"/>
@@
 <net name="IN" class="0">
 <segment>
-<pinref part="IN1" gate="G$1" pin="IN"/>
+<pinref part="IN" gate="G$1" pin="IN"/>
 <pinref part="R1" gate="G$1" pin="2"/>
 <wire x1="-5.08" y1="83.82" x2="0" y2="83.82" width="0.1524" layer="91"/>
@@
 <net name="+9V" class="0">
 <segment>
-<pinref part="+9V1" gate="+9V" pin="+9V"/>
+<pinref part="+9V" gate="+9V" pin="+9V"/>
 <pinref part="D2" gate="1" pin="A"/>
 <wire x1="-5.08" y1="68.58" x2="0" y2="68.58" width="0.1524" layer="91"/>
@@
 <net name="GND" class="0">
 <segment>
-<pinref part="GND1" gate="GND" pin="GND"/>
+<pinref part="GND" gate="GND" pin="GND"/>
 <pinref part="R4" gate="G$1" pin="1"/>
 <wire x1="12.7" y1="48.26" x2="12.7" y2="55.88" width="0.1524" layer="91"/>
@@
 <segment>
 <pinref part="VOL" gate="G$1" pin="2"/>
-<pinref part="OUT1" gate="G$1" pin="OUT"/>
+<pinref part="OUT" gate="G$1" pin="OUT"/>
 <wire x1="187.96" y1="48.26" x2="190.5" y2="48.26" width="0.1524" layer="91"/>
 </segment>
